Commit message: Increase lbr ik solver attempts, modify link_tool tf to accrount for ee change

File: src/tekkneeca/lbr_fri_ros2_stack/lbr_description/urdf/med7/med7_description.urdf.xacro (robot description, xacro)
@@ -317,5 +317,5 @@
             <parent link="link_drillbit" />
             <child link="link_tool" />
-            <origin xyz="0 0 0.031" rpy="0 0 0" />
+            <origin xyz="0 0 0.201" rpy="0 0 0" />
         </joint>
         <link name="link_tool">
